Commit message: refactor

File: arm_description/urdf/arm.xacro (robot description, xacro)
@@ -1,79 +1,6 @@
-<?xml version="1.0" ?>
+<?xml version="1.0"?>
 <robot name="arm" xmlns:xacro="http://www.ros.org/wiki/xacro">
-<xacro:include filename="$(find arm_description)/urdf/materials.xacro" />
-<xacro:include filename="$(find arm_description)/urdf/arm.trans" />
-<xacro:include filename="$(find arm_description)/urdf/arm.gazebo" />
-<link name="base_link">
-  <inertial>
-    <origin xyz="1.5731329451305026e-13 -2.543236304324506e-16 0.04811936745718893" rpy="0 0 0"/>
-    <mass value="0.15790854887087455"/>
-    <inertia ixx="0.000119" iyy="0.000119" izz="0.000201" ixy="0.0" iyz="-0.0" ixz="0.0"/>
-  </inertial>
-  <visual>
-    <origin xyz="0 0 0" rpy="0 0 0"/>
-    <geometry>
-      <mesh filename="file://$(find arm_description)/meshes/base_link.stl" scale="0.001 0.001 0.001"/>
-    </geometry>
-    <material name="silver"/>
-  </visual>
-  <collision>
-    <origin xyz="0 0 0" rpy="0 0 0"/>
-    <geometry>
-      <mesh filename="file://$(find arm_description)/meshes/base_link.stl" scale="0.001 0.001 0.001"/>
-    </geometry>
-  </collision>
-</link>
-<link name="shoulder_mount_1">
-  <inertial>
-    <origin xyz="5.144548699475028e-06 0.014758819360046764 0.01645492919069829" rpy="0 0 0"/>
-    <mass value="0.3050001457280305"/>
-    <inertia ixx="0.000394" iyy="0.00031" izz="0.000353" ixy="-0.0" iyz="-0.000104" ixz="-0.0"/>
-  </inertial>
-  <visual>
-    <origin xyz="-0.0 -0.0 -0.0531" rpy="0 0 0"/>
-    <geometry>
-      <mesh filename="file://$(find arm_description)/meshes/shoulder_mount_1.stl" scale="0.001 0.001 0.001"/>
-    </geometry>
-    <material name="silver"/>
-  </visual>
-  <collision>
-    <origin xyz="-0.0 -0.0 -0.0531" rpy="0 0 0"/>
-    <geometry>
-      <mesh filename="file://$(find arm_description)/meshes/shoulder_mount_1.stl" scale="0.001 0.001 0.001"/>
-    </geometry>
-  </collision>
-</link>
-<link name="shoulder_1">
-  <inertial>
-    <origin xyz="-0.059999999999999915 -0.004999999403953563 -2.7755575615628914e-17" rpy="0 0 0"/>
-    <mass value="0.9615034035508284"/>
-    <inertia ixx="0.00037" iyy="0.002872" izz="0.002518" ixy="0.0" iyz="-0.0" ixz="0.0"/>
-  </inertial>
-  <visual>
-    <origin xyz="0.0001 -0.035 -0.1162" rpy="0 0 0"/>
-    <geometry>
-      <mesh filename="file://$(find arm_description)/meshes/shoulder_1.stl" scale="0.001 0.001 0.001"/>
-    </geometry>
-    <material name="silver"/>
-  </visual>
-  <collision>
-    <origin xyz="0.0001 -0.035 -0.1162" rpy="0 0 0"/>
-    <geometry>
-      <mesh filename="file://$(find arm_description)/meshes/shoulder_1.stl" scale="0.001 0.001 0.001"/>
-    </geometry>
-  </collision>
-</link>
-<joint name="base_joint" type="continuous">
-  <origin xyz="0.0 0.0 0.0531" rpy="0 0 0"/>
-  <parent link="base_link"/>
-  <child link="shoulder_mount_1"/>
-  <axis xyz="0.0 0.0 1.0"/>
-</joint>
-<joint name="shoulder_joint" type="revolute">
-  <origin xyz="-0.0001 0.035 0.0631" rpy="0 0 0"/>
-  <parent link="shoulder_mount_1"/>
-  <child link="shoulder_1"/>
-  <axis xyz="0.0 1.0 0.0"/>
-  <limit upper="3.141593" lower="0.0" effort="100" velocity="100"/>
-</joint>
+    <xacro:arg name="is_sim" default="true"/>
+    <xacro:include filename="$(find arm_description)/urdf/arm.macro.xacro"/>
+    <xacro:arm is_sim="$is_sim"/>
 </robot>
