Commit message: gazebo control

File: arm_description/urdf/arm_core.xacro (robot description, xacro)
@@ -75,3 +75,9 @@
   <limit upper="3.141593" lower="0.0" effort="100" velocity="100"/>
 </joint>
+    <link name="world"/>
+    <joint name="world" type="fixed">
+        <parent link="world"/>
+        <child link="base_link"/>
+        <origin xyz="0 0 0" rpy="0 0 0"/>
+    </joint>
 </robot>

Commit message: refactor

File: arm_description/urdf/arm_core.xacro (robot description, xacro)
@@ -1,78 +1,78 @@
 <?xml version="1.0" ?>
 <robot name="arm" xmlns:xacro="http://www.ros.org/wiki/xacro">
-<xacro:include filename="$(find arm_description)/urdf/materials.xacro" />
-<link name="base_link">
-  <inertial>
-    <origin xyz="1.5731329451305026e-13 -2.543236304324506e-16 0.04811936745718893" rpy="0 0 0"/>
-    <mass value="0.15790854887087455"/>
-    <inertia ixx="0.000119" iyy="0.000119" izz="0.000201" ixy="0.0" iyz="-0.0" ixz="0.0"/>
-  </inertial>
-  <visual>
-    <origin xyz="0 0 0" rpy="0 0 0"/>
-    <geometry>
-      <mesh filename="file://$(find arm_description)/meshes/base_link.stl" scale="0.001 0.001 0.001"/>
-    </geometry>
-    <material name="silver"/>
-  </visual>
-  <collision>
-    <origin xyz="0 0 0" rpy="0 0 0"/>
-    <geometry>
-      <mesh filename="file://$(find arm_description)/meshes/base_link.stl" scale="0.001 0.001 0.001"/>
-    </geometry>
-  </collision>
-</link>
-<link name="shoulder_mount_1">
-  <inertial>
-    <origin xyz="5.144548699475028e-06 0.014758819360046764 0.01645492919069829" rpy="0 0 0"/>
-    <mass value="0.3050001457280305"/>
-    <inertia ixx="0.000394" iyy="0.00031" izz="0.000353" ixy="-0.0" iyz="-0.000104" ixz="-0.0"/>
-  </inertial>
-  <visual>
-    <origin xyz="-0.0 -0.0 -0.0531" rpy="0 0 0"/>
-    <geometry>
-      <mesh filename="file://$(find arm_description)/meshes/shoulder_mount_1.stl" scale="0.001 0.001 0.001"/>
-    </geometry>
-    <material name="silver"/>
-  </visual>
-  <collision>
-    <origin xyz="-0.0 -0.0 -0.0531" rpy="0 0 0"/>
-    <geometry>
-      <mesh filename="file://$(find arm_description)/meshes/shoulder_mount_1.stl" scale="0.001 0.001 0.001"/>
-    </geometry>
-  </collision>
-</link>
-<link name="shoulder_1">
-  <inertial>
-    <origin xyz="-0.059999999999999915 -0.004999999403953563 -2.7755575615628914e-17" rpy="0 0 0"/>
-    <mass value="0.9615034035508284"/>
-    <inertia ixx="0.00037" iyy="0.002872" izz="0.002518" ixy="0.0" iyz="-0.0" ixz="0.0"/>
-  </inertial>
-  <visual>
-    <origin xyz="0.0001 -0.035 -0.1162" rpy="0 0 0"/>
-    <geometry>
-      <mesh filename="file://$(find arm_description)/meshes/shoulder_1.stl" scale="0.001 0.001 0.001"/>
-    </geometry>
-    <material name="silver"/>
-  </visual>
-  <collision>
-    <origin xyz="0.0001 -0.035 -0.1162" rpy="0 0 0"/>
-    <geometry>
-      <mesh filename="file://$(find arm_description)/meshes/shoulder_1.stl" scale="0.001 0.001 0.001"/>
-    </geometry>
-  </collision>
-</link>
-<joint name="base_joint" type="continuous">
-  <origin xyz="0.0 0.0 0.0531" rpy="0 0 0"/>
-  <parent link="base_link"/>
-  <child link="shoulder_mount_1"/>
-  <axis xyz="0.0 0.0 1.0"/>
-</joint>
-<joint name="shoulder_joint" type="revolute">
-  <origin xyz="-0.0001 0.035 0.0631" rpy="0 0 0"/>
-  <parent link="shoulder_mount_1"/>
-  <child link="shoulder_1"/>
-  <axis xyz="0.0 1.0 0.0"/>
-  <limit upper="3.141593" lower="0.0" effort="100" velocity="100"/>
-</joint>
+    <xacro:include filename="$(find arm_description)/urdf/materials.xacro"/>
+    <link name="base_link">
+        <inertial>
+            <origin xyz="1.5731329451305026e-13 -2.543236304324506e-16 0.04811936745718893" rpy="0 0 0"/>
+            <mass value="0.15790854887087455"/>
+            <inertia ixx="0.000119" iyy="0.000119" izz="0.000201" ixy="0.0" iyz="-0.0" ixz="0.0"/>
+        </inertial>
+        <visual>
+            <origin xyz="0 0 0" rpy="0 0 0"/>
+            <geometry>
+                <mesh filename="file://$(find arm_description)/meshes/base_link.stl" scale="0.001 0.001 0.001"/>
+            </geometry>
+            <material name="silver"/>
+        </visual>
+        <collision>
+            <origin xyz="0 0 0" rpy="0 0 0"/>
+            <geometry>
+                <mesh filename="file://$(find arm_description)/meshes/base_link.stl" scale="0.001 0.001 0.001"/>
+            </geometry>
+        </collision>
+    </link>
+    <link name="shoulder_mount_1">
+        <inertial>
+            <origin xyz="5.144548699475028e-06 0.014758819360046764 0.01645492919069829" rpy="0 0 0"/>
+            <mass value="0.3050001457280305"/>
+            <inertia ixx="0.000394" iyy="0.00031" izz="0.000353" ixy="-0.0" iyz="-0.000104" ixz="-0.0"/>
+        </inertial>
+        <visual>
+            <origin xyz="-0.0 -0.0 -0.0531" rpy="0 0 0"/>
+            <geometry>
+                <mesh filename="file://$(find arm_description)/meshes/shoulder_mount_1.stl" scale="0.001 0.001 0.001"/>
+            </geometry>
+            <material name="silver"/>
+        </visual>
+        <collision>
+            <origin xyz="-0.0 -0.0 -0.0531" rpy="0 0 0"/>
+            <geometry>
+                <mesh filename="file://$(find arm_description)/meshes/shoulder_mount_1.stl" scale="0.001 0.001 0.001"/>
+            </geometry>
+        </collision>
+    </link>
+    <link name="shoulder_1">
+        <inertial>
+            <origin xyz="-0.059999999999999915 -0.004999999403953563 -2.7755575615628914e-17" rpy="0 0 0"/>
+            <mass value="0.9615034035508284"/>
+            <inertia ixx="0.00037" iyy="0.002872" izz="0.002518" ixy="0.0" iyz="-0.0" ixz="0.0"/>
+        </inertial>
+        <visual>
+            <origin xyz="0.0001 -0.035 -0.1162" rpy="0 0 0"/>
+            <geometry>
+                <mesh filename="file://$(find arm_description)/meshes/shoulder_1.stl" scale="0.001 0.001 0.001"/>
+            </geometry>
+            <material name="silver"/>
+        </visual>
+        <collision>
+            <origin xyz="0.0001 -0.035 -0.1162" rpy="0 0 0"/>
+            <geometry>
+                <mesh filename="file://$(find arm_description)/meshes/shoulder_1.stl" scale="0.001 0.001 0.001"/>
+            </geometry>
+        </collision>
+    </link>
+    <joint name="base_joint" type="continuous">
+        <origin xyz="0.0 0.0 0.0531" rpy="0 0 0"/>
+        <parent link="base_link"/>
+        <child link="shoulder_mount_1"/>
+        <axis xyz="0.0 0.0 1.0"/>
+    </joint>
+    <joint name="shoulder_joint" type="revolute">
+        <origin xyz="-0.0001 0.035 0.0631" rpy="0 0 0"/>
+        <parent link="shoulder_mount_1"/>
+        <child link="shoulder_1"/>
+        <axis xyz="0.0 1.0 0.0"/>
+        <limit upper="3.141593" lower="0.0" effort="100" velocity="100"/>
+    </joint>
     <link name="world"/>
     <joint name="world" type="fixed">

Commit message: -virtual_joint in urdf -removed VIRTUAL JOINT in srdf -updated rviz config -install.sh

File: arm_description/urdf/arm_core.xacro (robot description, xacro)
@@ -76,5 +76,5 @@
     </joint>
     <link name="world"/>
-    <joint name="world" type="fixed">
+    <joint name="virtual_joint" type="fixed">
         <parent link="world"/>
         <child link="base_link"/>

Commit message: -fixed by relaxing shoulder_joint and biceptricep_joint limits

File: arm_description/urdf/arm_core.xacro (robot description, xacro)
@@ -84,10 +84,10 @@
     <link name="biceptricep_forearm_link_1">
         <inertial>
-            <origin xyz="-0.06680915249598357 -0.009999999999999926 -8.604228440844963e-16" rpy="0 0 0"/>
+            <origin xyz="-0.06680915249598346 0.010000000000000002 6.661338147750939e-16" rpy="0 0 0"/>
             <mass value="2.4998312500297173"/>
-            <inertia ixx="0.001444" iyy="0.009664" izz="0.008376" ixy="0.0" iyz="-0.0" ixz="-0.0"/>
+            <inertia ixx="0.001444" iyy="0.009664" izz="0.008376" ixy="0.0" iyz="-0.0" ixz="0.0"/>
         </inertial>
         <visual>
-            <origin xyz="0.2 0.0775 -0.1625" rpy="0 0 0"/>
+            <origin xyz="0.2 -0.0375 -0.1625" rpy="0 0 0"/>
             <geometry>
                 <mesh filename="file://$(find arm_description)/meshes/biceptricep_forearm_link_1.stl" scale="0.001 0.001 0.001"/>
@@ -96,5 +96,5 @@
         </visual>
         <collision>
-            <origin xyz="0.2 0.0775 -0.1625" rpy="0 0 0"/>
+            <origin xyz="0.2 -0.0375 -0.1625" rpy="0 0 0"/>
             <geometry>
                 <mesh filename="file://$(find arm_description)/meshes/biceptricep_forearm_link_1.stl" scale="0.001 0.001 0.001"/>
@@ -104,10 +104,10 @@
     <link name="forearm_1">
         <inertial>
-            <origin xyz="0.0 -0.057499999999999926 -1.942890293094024e-16" rpy="0 0 0"/>
+            <origin xyz="0.0 0.0575 0.0" rpy="0 0 0"/>
             <mass value="5.122656437250909"/>
             <inertia ixx="0.007959" iyy="0.004626" izz="0.007959" ixy="-0.0" iyz="0.0" ixz="0.0"/>
         </inertial>
         <visual>
-            <origin xyz="0.4 0.0775 -0.1625" rpy="0 0 0"/>
+            <origin xyz="0.4 -0.0375 -0.1625" rpy="0 0 0"/>
             <geometry>
                 <mesh filename="file://$(find arm_description)/meshes/forearm_1.stl" scale="0.001 0.001 0.001"/>
@@ -116,5 +116,5 @@
         </visual>
         <collision>
-            <origin xyz="0.4 0.0775 -0.1625" rpy="0 0 0"/>
+            <origin xyz="0.4 -0.0375 -0.1625" rpy="0 0 0"/>
             <geometry>
                 <mesh filename="file://$(find arm_description)/meshes/forearm_1.stl" scale="0.001 0.001 0.001"/>
@@ -124,10 +124,10 @@
     <link name="wrist_1">
         <inertial>
-            <origin xyz="-1.6653345369377348e-16 -0.04673529188000056 -2.8160945797495174e-11" rpy="0 0 0"/>
+            <origin xyz="-1.1102230246251565e-16 0.04673529188000053 2.816077926404148e-11" rpy="0 0 0"/>
             <mass value="5.211945183934523"/>
-            <inertia ixx="0.008209" iyy="0.008038" izz="0.004805" ixy="-0.0" iyz="0.0" ixz="-0.0"/>
+            <inertia ixx="0.008209" iyy="0.008038" izz="0.004805" ixy="0.0" iyz="0.0" ixz="0.0"/>
         </inertial>
         <visual>
-            <origin xyz="0.4 0.1925 -0.1625" rpy="0 0 0"/>
+            <origin xyz="0.4 -0.1525 -0.1625" rpy="0 0 0"/>
             <geometry>
                 <mesh filename="file://$(find arm_description)/meshes/wrist_1.stl" scale="0.001 0.001 0.001"/>
@@ -136,5 +136,5 @@
         </visual>
         <collision>
-            <origin xyz="0.4 0.1925 -0.1625" rpy="0 0 0"/>
+            <origin xyz="0.4 -0.1525 -0.1625" rpy="0 0 0"/>
             <geometry>
                 <mesh filename="file://$(find arm_description)/meshes/wrist_1.stl" scale="0.001 0.001 0.001"/>
@@ -149,10 +149,10 @@
         <limit upper="6.265732" lower="0.0" effort="100" velocity="100"/>
     </joint>
-    <joint name="shoulder_joint" type="revolute">
+    <joint name="shoulder_joint" type="continuous">
         <origin xyz="0.0 -0.0575 0.0475" rpy="0 0 0"/>
         <parent link="shoulder_1"/>
         <child link="should_biceptricep_link_1"/>
         <axis xyz="0.0 -1.0 -0.0"/>
-        <limit upper="6.283185" lower="3.141593" effort="100" velocity="100"/>
+<!--        <limit upper="6.283185" lower="3.141593" effort="100" velocity="100"/>-->
     </joint>
     <joint name="Rigid 7" type="fixed">
@@ -161,10 +161,10 @@
         <child link="biceptricep_1"/>
     </joint>
-    <joint name="biceptricep_joint" type="revolute">
-        <origin xyz="0.0 0.0 0.0" rpy="0 0 0"/>
+    <joint name="biceptricep_joint" type="continuous">
+        <origin xyz="0.0 0.115 0.0" rpy="0 0 0"/>
         <parent link="biceptricep_1"/>
         <child link="biceptricep_forearm_link_1"/>
-        <axis xyz="0.0 -1.0 -0.0"/>
-        <limit upper="6.265732" lower="0.0" effort="100" velocity="100"/>
+        <axis xyz="0.0 1.0 0.0"/>
+<!--        <limit upper="6.265732" lower="0.0" effort="100" velocity="100"/>-->
     </joint>
     <joint name="Rigid 8" type="fixed">
@@ -174,8 +174,8 @@
     </joint>
     <joint name="forearm_joint" type="continuous">
-        <origin xyz="0.0 -0.115 0.0" rpy="0 0 0"/>
+        <origin xyz="0.0 0.115 0.0" rpy="0 0 0"/>
         <parent link="forearm_1"/>
         <child link="wrist_1"/>
-        <axis xyz="-0.0 1.0 -0.0"/>
+        <axis xyz="-0.0 -1.0 0.0"/>
     </joint>
     <link name="world"/>

Commit message: -limited shoulder_joint

File: arm_description/urdf/arm_core.xacro (robot description, xacro)
@@ -149,10 +149,10 @@
         <limit upper="6.265732" lower="0.0" effort="100" velocity="100"/>
     </joint>
-    <joint name="shoulder_joint" type="continuous">
+    <joint name="shoulder_joint" type="revolute">
         <origin xyz="0.0 -0.0575 0.0475" rpy="0 0 0"/>
         <parent link="shoulder_1"/>
         <child link="should_biceptricep_link_1"/>
         <axis xyz="0.0 -1.0 -0.0"/>
-<!--        <limit upper="6.283185" lower="3.141593" effort="100" velocity="100"/>-->
+        <limit upper="6.265732" lower="0.0" effort="100" velocity="100"/>
     </joint>
     <joint name="Rigid 7" type="fixed">

Commit message: -fixed joints' limits

File: arm_description/urdf/arm_core.xacro (robot description, xacro)
@@ -2,4 +2,7 @@
 <robot name="arm" xmlns:xacro="http://www.ros.org/wiki/xacro">
     <xacro:include filename="$(find arm_description)/urdf/materials.xacro"/>
+    <xacro:property name="PI" value="3.14159265359"/>
+    <xacro:property name="effort" value="30"/>
+    <xacro:property name="velocity" value="10"/>
     <link name="base_link">
         <inertial>
@@ -51,5 +54,6 @@
             <origin xyz="-0.0 0.0575 -0.1625" rpy="0 0 0"/>
             <geometry>
-                <mesh filename="file://$(find arm_description)/meshes/should_biceptricep_link_1.stl" scale="0.001 0.001 0.001"/>
+                <mesh filename="file://$(find arm_description)/meshes/should_biceptricep_link_1.stl"
+                      scale="0.001 0.001 0.001"/>
             </geometry>
             <material name="silver"/>
@@ -58,5 +62,6 @@
             <origin xyz="-0.0 0.0575 -0.1625" rpy="0 0 0"/>
             <geometry>
-                <mesh filename="file://$(find arm_description)/meshes/should_biceptricep_link_1.stl" scale="0.001 0.001 0.001"/>
+                <mesh filename="file://$(find arm_description)/meshes/should_biceptricep_link_1.stl"
+                      scale="0.001 0.001 0.001"/>
             </geometry>
         </collision>
@@ -91,5 +96,6 @@
             <origin xyz="0.2 -0.0375 -0.1625" rpy="0 0 0"/>
             <geometry>
-                <mesh filename="file://$(find arm_description)/meshes/biceptricep_forearm_link_1.stl" scale="0.001 0.001 0.001"/>
+                <mesh filename="file://$(find arm_description)/meshes/biceptricep_forearm_link_1.stl"
+                      scale="0.001 0.001 0.001"/>
             </geometry>
             <material name="silver"/>
@@ -98,5 +104,6 @@
             <origin xyz="0.2 -0.0375 -0.1625" rpy="0 0 0"/>
             <geometry>
-                <mesh filename="file://$(find arm_description)/meshes/biceptricep_forearm_link_1.stl" scale="0.001 0.001 0.001"/>
+                <mesh filename="file://$(find arm_description)/meshes/biceptricep_forearm_link_1.stl"
+                      scale="0.001 0.001 0.001"/>
             </geometry>
         </collision>
@@ -147,5 +154,5 @@
         <child link="shoulder_1"/>
         <axis xyz="0.0 0.0 1.0"/>
-        <limit upper="6.265732" lower="0.0" effort="100" velocity="100"/>
+        <limit lower="-${PI/2}" upper="${PI/2}" effort="${effort}" velocity="${velocity}"/>
     </joint>
     <joint name="shoulder_joint" type="revolute">
@@ -154,5 +161,5 @@
         <child link="should_biceptricep_link_1"/>
         <axis xyz="0.0 -1.0 -0.0"/>
-        <limit upper="6.265732" lower="0.0" effort="100" velocity="100"/>
+        <limit lower="-${PI/2}" upper="${PI/2}" effort="${effort}" velocity="${velocity}"/>
     </joint>
     <joint name="Rigid 7" type="fixed">
@@ -161,10 +168,10 @@
         <child link="biceptricep_1"/>
     </joint>
-    <joint name="biceptricep_joint" type="continuous">
+    <joint name="biceptricep_joint" type="revolute">
         <origin xyz="0.0 0.115 0.0" rpy="0 0 0"/>
         <parent link="biceptricep_1"/>
         <child link="biceptricep_forearm_link_1"/>
         <axis xyz="0.0 1.0 0.0"/>
-<!--        <limit upper="6.265732" lower="0.0" effort="100" velocity="100"/>-->
+        <limit lower="-${PI/2}" upper="${PI/2}" effort="${effort}" velocity="${velocity}"/>
     </joint>
     <joint name="Rigid 8" type="fixed">

Commit message: -made forearm revolute with limits -updated rviz config with Trajectory & PlanningScene

File: arm_description/urdf/arm_core.xacro (robot description, xacro)
@@ -180,9 +180,10 @@
         <child link="forearm_1"/>
     </joint>
-    <joint name="forearm_joint" type="continuous">
+    <joint name="forearm_joint" type="revolute">
         <origin xyz="0.0 0.115 0.0" rpy="0 0 0"/>
         <parent link="forearm_1"/>
         <child link="wrist_1"/>
         <axis xyz="-0.0 -1.0 0.0"/>
+        <limit lower="-${PI/2}" upper="${PI/2}" effort="${effort}" velocity="${velocity}"/>
     </joint>
     <link name="world"/>

Commit message: -updated joints' limits

File: arm_description/urdf/arm_core.xacro (robot description, xacro)
@@ -161,5 +161,5 @@
         <child link="should_biceptricep_link_1"/>
         <axis xyz="0.0 -1.0 -0.0"/>
-        <limit lower="-${PI/2}" upper="${PI/2}" effort="${effort}" velocity="${velocity}"/>
+        <limit lower="-${PI}" upper="0" effort="${effort}" velocity="${velocity}"/>
     </joint>
     <joint name="Rigid 7" type="fixed">
@@ -173,5 +173,5 @@
         <child link="biceptricep_forearm_link_1"/>
         <axis xyz="0.0 1.0 0.0"/>
-        <limit lower="-${PI/2}" upper="${PI/2}" effort="${effort}" velocity="${velocity}"/>
+        <limit lower="0" upper="${PI}" effort="${effort}" velocity="${velocity}"/>
     </joint>
     <joint name="Rigid 8" type="fixed">
@@ -185,5 +185,5 @@
         <child link="wrist_1"/>
         <axis xyz="-0.0 -1.0 0.0"/>
-        <limit lower="-${PI/2}" upper="${PI/2}" effort="${effort}" velocity="${velocity}"/>
+        <limit lower="-${PI}" upper="${PI}" effort="${effort}" velocity="${velocity}"/>
     </joint>
     <link name="world"/>

Commit message: -increased range for waist_joint & shoulder_joint

File: arm_description/urdf/arm_core.xacro (robot description, xacro)
@@ -154,5 +154,5 @@
         <child link="shoulder_1"/>
         <axis xyz="0.0 0.0 1.0"/>
-        <limit lower="-${PI/2}" upper="${PI/2}" effort="${effort}" velocity="${velocity}"/>
+        <limit lower="-${PI}" upper="${PI}" effort="${effort}" velocity="${velocity}"/>
     </joint>
     <joint name="shoulder_joint" type="revolute">
@@ -173,5 +173,5 @@
         <child link="biceptricep_forearm_link_1"/>
         <axis xyz="0.0 1.0 0.0"/>
-        <limit lower="0" upper="${PI}" effort="${effort}" velocity="${velocity}"/>
+        <limit lower="-${PI}" upper="${PI}" effort="${effort}" velocity="${velocity}"/>
     </joint>
     <joint name="Rigid 8" type="fixed">
