Commit message: -changed links' names + panda_joint8

File: arm_description/urdf/arm_core.xacro (robot description, xacro)
@@ -25,5 +25,5 @@
         </collision>
     </link>
-    <link name="aa_1_1">
+    <link name="arm_link2_1">
         <inertial>
             <origin xyz="1.5654448004331833e-05 -0.02828101362582021 0.05185557651992784" rpy="0 0 0"/>
@@ -34,5 +34,5 @@
             <origin xyz="-0.0 -0.0 -0.1" rpy="0 0 0"/>
             <geometry>
-                <mesh filename="file://$(find arm_description)/meshes/aa_1_1.stl" scale="0.001 0.001 0.001"/>
+                <mesh filename="file://$(find arm_description)/meshes/arm_link2_1.stl" scale="0.001 0.001 0.001"/>
             </geometry>
             <material name="silver"/>
@@ -41,9 +41,9 @@
             <origin xyz="-0.0 -0.0 -0.1" rpy="0 0 0"/>
             <geometry>
-                <mesh filename="file://$(find arm_description)/meshes/aa_1_1.stl" scale="0.001 0.001 0.001"/>
-            </geometry>
-        </collision>
-    </link>
-    <link name="bb_1_1">
+                <mesh filename="file://$(find arm_description)/meshes/arm_link2_1.stl" scale="0.001 0.001 0.001"/>
+            </geometry>
+        </collision>
+    </link>
+    <link name="arm_link3_1">
         <inertial>
             <origin xyz="-0.00019632988035193946 0.006345060504398406 0.09901048510996069" rpy="0 0 0"/>
@@ -54,5 +54,5 @@
             <origin xyz="-1.8e-05 0.003 -0.160821" rpy="0 0 0"/>
             <geometry>
-                <mesh filename="file://$(find arm_description)/meshes/bb_1_1.stl" scale="0.001 0.001 0.001"/>
+                <mesh filename="file://$(find arm_description)/meshes/arm_link3_1.stl" scale="0.001 0.001 0.001"/>
             </geometry>
             <material name="silver"/>
@@ -61,9 +61,9 @@
             <origin xyz="-1.8e-05 0.003 -0.160821" rpy="0 0 0"/>
             <geometry>
-                <mesh filename="file://$(find arm_description)/meshes/bb_1_1.stl" scale="0.001 0.001 0.001"/>
-            </geometry>
-        </collision>
-    </link>
-    <link name="aa_2_1">
+                <mesh filename="file://$(find arm_description)/meshes/arm_link3_1.stl" scale="0.001 0.001 0.001"/>
+            </geometry>
+        </collision>
+    </link>
+    <link name="arm_link4_1">
         <inertial>
             <origin xyz="1.576364303761414e-05 -0.028281109488109926 0.05185557651992889" rpy="0 0 0"/>
@@ -74,5 +74,5 @@
             <origin xyz="0.000204 -0.000204 -0.313" rpy="0 0 0"/>
             <geometry>
-                <mesh filename="file://$(find arm_description)/meshes/aa_2_1.stl" scale="0.001 0.001 0.001"/>
+                <mesh filename="file://$(find arm_description)/meshes/arm_link4_1.stl" scale="0.001 0.001 0.001"/>
             </geometry>
             <material name="silver"/>
@@ -81,9 +81,9 @@
             <origin xyz="0.000204 -0.000204 -0.313" rpy="0 0 0"/>
             <geometry>
-                <mesh filename="file://$(find arm_description)/meshes/aa_2_1.stl" scale="0.001 0.001 0.001"/>
-            </geometry>
-        </collision>
-    </link>
-    <link name="bb_2_1">
+                <mesh filename="file://$(find arm_description)/meshes/arm_link4_1.stl" scale="0.001 0.001 0.001"/>
+            </geometry>
+        </collision>
+    </link>
+    <link name="arm_link5_1">
         <inertial>
             <origin xyz="-0.00019622068531865714 0.006344964642108612 0.09901048510996169" rpy="0 0 0"/>
@@ -94,5 +94,5 @@
             <origin xyz="0.000186 0.002796 -0.373821" rpy="0 0 0"/>
             <geometry>
-                <mesh filename="file://$(find arm_description)/meshes/bb_2_1.stl" scale="0.001 0.001 0.001"/>
+                <mesh filename="file://$(find arm_description)/meshes/arm_link5_1.stl" scale="0.001 0.001 0.001"/>
             </geometry>
             <material name="silver"/>
@@ -101,9 +101,9 @@
             <origin xyz="0.000186 0.002796 -0.373821" rpy="0 0 0"/>
             <geometry>
-                <mesh filename="file://$(find arm_description)/meshes/bb_2_1.stl" scale="0.001 0.001 0.001"/>
-            </geometry>
-        </collision>
-    </link>
-    <link name="Actuator_Cover_v4_1">
+                <mesh filename="file://$(find arm_description)/meshes/arm_link5_1.stl" scale="0.001 0.001 0.001"/>
+            </geometry>
+        </collision>
+    </link>
+    <link name="arm_link6_1">
         <inertial>
             <origin xyz="2.183900666265855e-07 -1.917245794849252e-07 0.005955315753380375" rpy="0 0 0"/>
@@ -114,5 +114,5 @@
             <origin xyz="0.000408 -0.000408 -0.526" rpy="0 0 0"/>
             <geometry>
-                <mesh filename="file://$(find arm_description)/meshes/Actuator_Cover_v4_1.stl" scale="0.001 0.001 0.001"/>
+                <mesh filename="file://$(find arm_description)/meshes/arm_link6_1.stl" scale="0.001 0.001 0.001"/>
             </geometry>
             <material name="silver"/>
@@ -121,5 +121,5 @@
             <origin xyz="0.000408 -0.000408 -0.526" rpy="0 0 0"/>
             <geometry>
-                <mesh filename="file://$(find arm_description)/meshes/Actuator_Cover_v4_1.stl" scale="0.001 0.001 0.001"/>
+                <mesh filename="file://$(find arm_description)/meshes/arm_link6_1.stl" scale="0.001 0.001 0.001"/>
             </geometry>
         </collision>
@@ -168,5 +168,5 @@
         <origin xyz="0.0 0.0 0.1" rpy="0 0 0"/>
         <parent link="base_link"/>
-        <child link="aa_1_1"/>
+        <child link="arm_link2_1"/>
         <axis xyz="0.0 0.0 1.0"/>
         <limit lower="-${PI}" upper="${PI}" effort="${effort}" velocity="${velocity}"/>
@@ -174,6 +174,6 @@
     <joint name="shoulder_joint" type="revolute">
         <origin xyz="1.8e-05 -0.003 0.060821" rpy="0 0 0"/>
-        <parent link="aa_1_1"/>
-        <child link="bb_1_1"/>
+        <parent link="arm_link2_1"/>
+        <child link="arm_link3_1"/>
         <axis xyz="0.0 1.0 0.0"/>
         <limit lower="-1.833" upper="1.833" effort="${effort}" velocity="${velocity}"/>
@@ -181,6 +181,6 @@
     <joint name="biceptricep_joint" type="revolute">
         <origin xyz="-0.000222 0.003204 0.152179" rpy="0 0 0"/>
-        <parent link="bb_1_1"/>
-        <child link="aa_2_1"/>
+        <parent link="arm_link3_1"/>
+        <child link="arm_link4_1"/>
         <axis xyz="0.0 -0.0 1.0"/>
         <limit lower="-${PI}" upper="${PI}" effort="${effort}" velocity="${velocity}"/>
@@ -188,6 +188,6 @@
     <joint name="forearm_joint" type="revolute">
         <origin xyz="1.8e-05 -0.003 0.060821" rpy="0 0 0"/>
-        <parent link="aa_2_1"/>
-        <child link="bb_2_1"/>
+        <parent link="arm_link4_1"/>
+        <child link="arm_link5_1"/>
         <axis xyz="0.0 1.0 0.0"/>
         <limit lower="-1.833" upper="1.833" effort="${effort}" velocity="${velocity}"/>
@@ -195,12 +195,19 @@
     <joint name="wrist_joint" type="revolute">
         <origin xyz="-0.000222 0.003204 0.152179" rpy="0 0 0"/>
-        <parent link="bb_2_1"/>
-        <child link="Actuator_Cover_v4_1"/>
+        <parent link="arm_link5_1"/>
+        <child link="arm_link6_1"/>
         <axis xyz="0.0 -0.0 1.0"/>
         <limit lower="-${PI}" upper="${PI}" effort="${effort}" velocity="${velocity}"/>
     </joint>
+    <link name="panda_link8" />
+    <joint name="panda_joint8" type="fixed">
+        <origin rpy="0 0 0" xyz="0 0 0.107" />
+        <parent link="arm_link5_1" />
+        <child link="panda_link8" />
+        <axis xyz="0 0 0" />
+    </joint>
     <joint name="hand_joint" type="fixed">
         <origin xyz="0.0 0.0 0.0105" rpy="0 0 0"/>
-        <parent link="Actuator_Cover_v4_1"/>
+        <parent link="panda_link8"/>
         <child link="hand_1"/>
     </joint>
@@ -210,5 +217,5 @@
         <child link="finger_1"/>
         <axis xyz="0.0 -1.0 -0.0"/>
-        <limit lower="-0.09" upper="0.0" effort="100" velocity="100"/>
+        <limit upper="0.0" lower="-0.09" effort="100" velocity="100"/>
     </joint>
 </robot>

Commit message: updated description

File: arm_description/urdf/arm_core.xacro (robot description, xacro)
@@ -1,93 +1,81 @@
-<?xml version="1.0"?>
+<?xml version="1.0" ?>
 <robot name="arm" xmlns:xacro="http://www.ros.org/wiki/xacro">
-  <xacro:property name="PI" value="3.14159265359" />
-  <xacro:property name="effort" value="30" />
-  <xacro:property name="velocity" value="10" />
-  <material name="black">
-    <color rgba="0 0 0 1" />
-</material>
-  <link name="world" />
-  <link name="base_link">
-    <inertial>
-      <origin xyz="-8.003962236693073e-05 -6.3633345680673e-06 -0.0902510859444478" rpy="0 0 0" />
-      <mass value="13.209210477237487" />
-      <inertia ixx="0.022854" iyy="0.037448" izz="0.042454" ixy="0.0" iyz="-0.0" ixz="-7e-06" />
-    </inertial>
-    <visual>
-      <origin xyz="0 0 0" rpy="0 0 0" />
-      <geometry>
-        <mesh filename="file://$(find arm_description)/meshes/base_link.stl"
-          scale="0.001 0.001 0.001" />
-      </geometry>
-      <material name="black" />
-    </visual>
-    <collision>
-      <origin xyz="0 0 0" rpy="0 0 0" />
-      <geometry>
-        <mesh filename="file://$(find arm_description)/meshes/base_link.stl"
-          scale="0.001 0.001 0.001" />
-      </geometry>
-    </collision>
-  </link>
-  <!-- base_joint fixes base_link to the environment -->
-  <joint name="base_joint" type="fixed">
-    <parent link="world" />
-    <child link="base_link" />
-    <origin xyz="0 0 0" rpy="0 0 0" />
-    <axis xyz="0 0 1" />
-  </joint>
-  <link name="j2">
-    <inertial>
-      <origin xyz="-4.995526395401573e-05 0.08189630150884797 0.11003474433619179" rpy="0 0 0" />
-      <mass value="13.236708010334862" />
-      <inertia ixx="0.037769" iyy="0.042685" izz="0.022945" ixy="0.0" iyz="-0.000135" ixz="0.0" />
-    </inertial>
-    <visual>
-      <origin xyz="-0.02925 -4.4e-05 0.04332" rpy="0 0 0" />
-      <geometry>
-        <mesh filename="file://$(find arm_description)/meshes/j2.stl" scale="0.001 0.001 0.001" />
-      </geometry>
-      <material name="black" />
-    </visual>
-    <collision>
-      <origin xyz="-0.02925 -4.4e-05 0.04332" rpy="0 0 0" />
-      <geometry>
-        <mesh filename="file://$(find arm_description)/meshes/j2.stl" scale="0.001 0.001 0.001" />
-      </geometry>
-    </collision>
-  </link>
-  <link name="j3">
-    <inertial>
-      <origin xyz="-0.10862594613593025 -0.05360196950323787 -4.739058210631586e-05" rpy="0 0 0" />
-      <mass value="6.378639750773571" />
-      <inertia ixx="0.009134" iyy="0.007444" izz="0.010645" ixy="-0.000109" iyz="-0.0" ixz="-0.0" />
-    </inertial>
-    <visual>
-      <origin xyz="-0.02915 -0.035125 -0.09623" rpy="0 0 0" />
-      <geometry>
-        <mesh filename="file://$(find arm_description)/meshes/j3.stl" scale="0.001 0.001 0.001" />
-      </geometry>
-      <material name="black" />
-    </visual>
-    <collision>
-      <origin xyz="-0.02915 -0.035125 -0.09623" rpy="0 0 0" />
-      <geometry>
-        <mesh filename="file://$(find arm_description)/meshes/j3.stl" scale="0.001 0.001 0.001" />
-      </geometry>
-    </collision>
-  </link>
-  <joint name="joint_1" type="revolute">
-    <origin xyz="0.02925 4.4e-05 -0.04332" rpy="0 0 0" />
-    <parent link="base_link" />
-    <child link="j2" />
-    <axis xyz="0.0 0.0 -1.0" />
-    <limit upper="6.265732" lower="0.0" effort="${effort}" velocity="${velocity}"  />
-  </joint>
-  <joint name="joint_2" type="revolute">
-    <origin xyz="-0.0001 0.035081 0.13955" rpy="0 0 0" />
-    <parent link="j2" />
-    <child link="j3" />
-    <axis xyz="0.0 1.0 0.0" />
-    <limit upper="3.141593" lower="0.0" effort="${effort}" velocity="${velocity}"  />
-  </joint>
+<xacro:include filename="$(find arm_description)/urdf/materials.xacro" />
+<xacro:property name="PI" value="3.14159265359" />
+<xacro:property name="effort" value="30" />
+<xacro:property name="velocity" value="10" />
+<link name="base_link">
+  <inertial>
+    <origin xyz="-8.003962236693073e-05 -6.3633345680673e-06 -0.0902510859444478" rpy="0 0 0"/>
+    <mass value="13.209210477237487"/>
+    <inertia ixx="0.022854" iyy="0.037448" izz="0.042454" ixy="0.0" iyz="-0.0" ixz="-7e-06"/>
+  </inertial>
+  <visual>
+    <origin xyz="0 0 0" rpy="0 0 0"/>
+    <geometry>
+      <mesh filename="file://$(find arm_description)/meshes/base_link.stl" scale="0.001 0.001 0.001"/>
+    </geometry>
+    <material name="silver"/>
+  </visual>
+  <collision>
+    <origin xyz="0 0 0" rpy="0 0 0"/>
+    <geometry>
+      <mesh filename="file://$(find arm_description)/meshes/base_link.stl" scale="0.001 0.001 0.001"/>
+    </geometry>
+  </collision>
+</link>
+<link name="j2_1">
+  <inertial>
+    <origin xyz="-4.995526395401573e-05 0.08189630150884797 0.11003474433619179" rpy="0 0 0"/>
+    <mass value="13.236708010334862"/>
+    <inertia ixx="0.037769" iyy="0.042685" izz="0.022945" ixy="0.0" iyz="-0.000135" ixz="0.0"/>
+  </inertial>
+  <visual>
+    <origin xyz="-0.02925 -4.4e-05 0.04332" rpy="0 0 0"/>
+    <geometry>
+      <mesh filename="file://$(find arm_description)/meshes/j2_1.stl" scale="0.001 0.001 0.001"/>
+    </geometry>
+    <material name="silver"/>
+  </visual>
+  <collision>
+    <origin xyz="-0.02925 -4.4e-05 0.04332" rpy="0 0 0"/>
+    <geometry>
+      <mesh filename="file://$(find arm_description)/meshes/j2_1.stl" scale="0.001 0.001 0.001"/>
+    </geometry>
+  </collision>
+</link>
+<link name="j3_1">
+  <inertial>
+    <origin xyz="-0.10862594613593025 -0.05360196950323787 -4.739058210631586e-05" rpy="0 0 0"/>
+    <mass value="6.378639750773571"/>
+    <inertia ixx="0.009134" iyy="0.007444" izz="0.010645" ixy="-0.000109" iyz="-0.0" ixz="-0.0"/>
+  </inertial>
+  <visual>
+    <origin xyz="-0.02915 -0.035125 -0.09623" rpy="0 0 0"/>
+    <geometry>
+      <mesh filename="file://$(find arm_description)/meshes/j3_1.stl" scale="0.001 0.001 0.001"/>
+    </geometry>
+    <material name="silver"/>
+  </visual>
+  <collision>
+    <origin xyz="-0.02915 -0.035125 -0.09623" rpy="0 0 0"/>
+    <geometry>
+      <mesh filename="file://$(find arm_description)/meshes/j3_1.stl" scale="0.001 0.001 0.001"/>
+    </geometry>
+  </collision>
+</link>
+<joint name="j1_j2" type="revolute">
+  <origin xyz="0.02925 4.4e-05 -0.04332" rpy="0 0 0"/>
+  <parent link="base_link"/>
+  <child link="j2_1"/>
+  <axis xyz="0.0 0.0 -1.0"/>
+  <limit upper="6.265732" lower="0.0" effort="${effort}" velocity="${velocity}"/>
+</joint>
+<joint name="j2_j3" type="revolute">
+  <origin xyz="-0.0001 0.035081 0.13955" rpy="0 0 0"/>
+  <parent link="j2_1"/>
+  <child link="j3_1"/>
+  <axis xyz="0.0 1.0 0.0"/>
+  <limit upper="3.141593" lower="0.0" effort="${effort}" velocity="${velocity}"/>
+</joint>
 </robot>

Commit message: setup assistant

File: arm_description/urdf/arm_core.xacro (robot description, xacro)
@@ -9,5 +9,4 @@
       <origin xyz="-3.761553966664625e-05 -0.1220000846362575 -0.1959085967473651" rpy="0 0 0" />
       <mass value="13.228344600133466" />
-      <inertia ixx="0.022903" iyy="0.037514" izz="0.042472" ixy="0.0" iyz="-0.0" ixz="-3.5e-05" />
     </inertial>
     <visual>
@@ -27,4 +26,9 @@
     </collision>
   </link>
+  <link name="world" />
+  <joint name="world_to_base" type="fixed">
+    <parent link="world" />
+    <child link="base_link" />
+  </joint>
   <link name="j1_1">
     <inertial>

Commit message: added inertia back

File: arm_description/urdf/arm_core.xacro (robot description, xacro)
@@ -9,4 +9,5 @@
       <origin xyz="-3.761553966664625e-05 -0.1220000846362575 -0.1959085967473651" rpy="0 0 0" />
       <mass value="13.228344600133466" />
+      <inertia ixx="0.022903" iyy="0.037514" izz="0.042472" ixy="0.0" iyz="-0.0" ixz="-3.5e-05" />
     </inertial>
     <visual>
