Commit message: -4 dof

File: arm_control/urdf/joints.macro.xacro (robot description, xacro)
@@ -2,5 +2,5 @@
 <robot xmlns:xacro="http://www.ros.org/wiki/xacro">
     <xacro:macro name="joints">
-        <joint name="base_joint">
+        <joint name="waist_joint">
             <command_interface name="position"/>
             <state_interface name="position">
@@ -14,4 +14,16 @@
             </state_interface>
         </joint>
+        <joint name="biceptricep_joint">
+            <command_interface name="position"/>
+            <state_interface name="position">
+                <param name="initial_value">0.0</param>
+            </state_interface>
+        </joint>
+        <joint name="forearm_joint">
+            <command_interface name="position"/>
+            <state_interface name="position">
+                <param name="initial_value">0.0</param>
+            </state_interface>
+        </joint>
     </xacro:macro>
 </robot>

File: arm_description/urdf/arm_core.xacro (robot description, xacro)
@@ -4,7 +4,7 @@
     <link name="base_link">
         <inertial>
-            <origin xyz="1.5731329451305026e-13 -2.543236304324506e-16 0.04811936745718893" rpy="0 0 0"/>
-            <mass value="0.15790854887087455"/>
-            <inertia ixx="0.000119" iyy="0.000119" izz="0.000201" ixy="0.0" iyz="-0.0" ixz="0.0"/>
+            <origin xyz="0.0 0.0 0.057499999999999975" rpy="0 0 0"/>
+            <mass value="5.122656437250909"/>
+            <inertia ixx="0.007959" iyy="0.007959" izz="0.004626" ixy="-0.0" iyz="0.0" ixz="0.0"/>
         </inertial>
         <visual>
@@ -22,32 +22,12 @@
         </collision>
     </link>
-    <link name="shoulder_mount_1">
+    <link name="shoulder_1">
         <inertial>
-            <origin xyz="5.144548699475028e-06 0.014758819360046764 0.01645492919069829" rpy="0 0 0"/>
-            <mass value="0.3050001457280305"/>
-            <inertia ixx="0.000394" iyy="0.00031" izz="0.000353" ixy="-0.0" iyz="-0.000104" ixz="-0.0"/>
+            <origin xyz="6.8492023198216155e-18 -2.816067379285414e-11 0.0467352918800006" rpy="0 0 0"/>
+            <mass value="5.211945183934523"/>
+            <inertia ixx="0.008209" iyy="0.004805" izz="0.008038" ixy="-0.0" iyz="-0.0" ixz="-0.0"/>
         </inertial>
         <visual>
-            <origin xyz="-0.0 -0.0 -0.0531" rpy="0 0 0"/>
-            <geometry>
-                <mesh filename="file://$(find arm_description)/meshes/shoulder_mount_1.stl" scale="0.001 0.001 0.001"/>
-            </geometry>
-            <material name="silver"/>
-        </visual>
-        <collision>
-            <origin xyz="-0.0 -0.0 -0.0531" rpy="0 0 0"/>
-            <geometry>
-                <mesh filename="file://$(find arm_description)/meshes/shoulder_mount_1.stl" scale="0.001 0.001 0.001"/>
-            </geometry>
-        </collision>
-    </link>
-    <link name="shoulder_1">
-        <inertial>
-            <origin xyz="-0.059999999999999915 -0.004999999403953563 -2.7755575615628914e-17" rpy="0 0 0"/>
-            <mass value="0.9615034035508284"/>
-            <inertia ixx="0.00037" iyy="0.002872" izz="0.002518" ixy="0.0" iyz="-0.0" ixz="0.0"/>
-        </inertial>
-        <visual>
-            <origin xyz="0.0001 -0.035 -0.1162" rpy="0 0 0"/>
+            <origin xyz="-0.0 -0.0 -0.115" rpy="0 0 0"/>
             <geometry>
                 <mesh filename="file://$(find arm_description)/meshes/shoulder_1.stl" scale="0.001 0.001 0.001"/>
@@ -56,5 +36,5 @@
         </visual>
         <collision>
-            <origin xyz="0.0001 -0.035 -0.1162" rpy="0 0 0"/>
+            <origin xyz="-0.0 -0.0 -0.115" rpy="0 0 0"/>
             <geometry>
                 <mesh filename="file://$(find arm_description)/meshes/shoulder_1.stl" scale="0.001 0.001 0.001"/>
@@ -62,16 +42,140 @@
         </collision>
     </link>
-    <joint name="base_joint" type="continuous">
-        <origin xyz="0.0 0.0 0.0531" rpy="0 0 0"/>
+    <link name="should_biceptricep_link_1">
+        <inertial>
+            <origin xyz="-0.06680915249598346 -0.009999999999999933 -8.326672684688674e-16" rpy="0 0 0"/>
+            <mass value="2.4998312500297173"/>
+            <inertia ixx="0.001444" iyy="0.009664" izz="0.008376" ixy="0.0" iyz="0.0" ixz="-0.0"/>
+        </inertial>
+        <visual>
+            <origin xyz="-0.0 0.0575 -0.1625" rpy="0 0 0"/>
+            <geometry>
+                <mesh filename="file://$(find arm_description)/meshes/should_biceptricep_link_1.stl" scale="0.001 0.001 0.001"/>
+            </geometry>
+            <material name="silver"/>
+        </visual>
+        <collision>
+            <origin xyz="-0.0 0.0575 -0.1625" rpy="0 0 0"/>
+            <geometry>
+                <mesh filename="file://$(find arm_description)/meshes/should_biceptricep_link_1.stl" scale="0.001 0.001 0.001"/>
+            </geometry>
+        </collision>
+    </link>
+    <link name="biceptricep_1">
+        <inertial>
+            <origin xyz="1.1102230246251565e-16 0.057500000000000065 -8.326672684688674e-17" rpy="0 0 0"/>
+            <mass value="5.122656437250909"/>
+            <inertia ixx="0.007959" iyy="0.004626" izz="0.007959" ixy="-0.0" iyz="0.0" ixz="0.0"/>
+        </inertial>
+        <visual>
+            <origin xyz="0.2 0.0775 -0.1625" rpy="0 0 0"/>
+            <geometry>
+                <mesh filename="file://$(find arm_description)/meshes/biceptricep_1.stl" scale="0.001 0.001 0.001"/>
+            </geometry>
+            <material name="silver"/>
+        </visual>
+        <collision>
+            <origin xyz="0.2 0.0775 -0.1625" rpy="0 0 0"/>
+            <geometry>
+                <mesh filename="file://$(find arm_description)/meshes/biceptricep_1.stl" scale="0.001 0.001 0.001"/>
+            </geometry>
+        </collision>
+    </link>
+    <link name="biceptricep_forearm_link_1">
+        <inertial>
+            <origin xyz="-0.06680915249598357 -0.009999999999999926 -8.604228440844963e-16" rpy="0 0 0"/>
+            <mass value="2.4998312500297173"/>
+            <inertia ixx="0.001444" iyy="0.009664" izz="0.008376" ixy="0.0" iyz="-0.0" ixz="-0.0"/>
+        </inertial>
+        <visual>
+            <origin xyz="0.2 0.0775 -0.1625" rpy="0 0 0"/>
+            <geometry>
+                <mesh filename="file://$(find arm_description)/meshes/biceptricep_forearm_link_1.stl" scale="0.001 0.001 0.001"/>
+            </geometry>
+            <material name="silver"/>
+        </visual>
+        <collision>
+            <origin xyz="0.2 0.0775 -0.1625" rpy="0 0 0"/>
+            <geometry>
+                <mesh filename="file://$(find arm_description)/meshes/biceptricep_forearm_link_1.stl" scale="0.001 0.001 0.001"/>
+            </geometry>
+        </collision>
+    </link>
+    <link name="forearm_1">
+        <inertial>
+            <origin xyz="0.0 -0.057499999999999926 -1.942890293094024e-16" rpy="0 0 0"/>
+            <mass value="5.122656437250909"/>
+            <inertia ixx="0.007959" iyy="0.004626" izz="0.007959" ixy="-0.0" iyz="0.0" ixz="0.0"/>
+        </inertial>
+        <visual>
+            <origin xyz="0.4 0.0775 -0.1625" rpy="0 0 0"/>
+            <geometry>
+                <mesh filename="file://$(find arm_description)/meshes/forearm_1.stl" scale="0.001 0.001 0.001"/>
+            </geometry>
+            <material name="silver"/>
+        </visual>
+        <collision>
+            <origin xyz="0.4 0.0775 -0.1625" rpy="0 0 0"/>
+            <geometry>
+                <mesh filename="file://$(find arm_description)/meshes/forearm_1.stl" scale="0.001 0.001 0.001"/>
+            </geometry>
+        </collision>
+    </link>
+    <link name="wrist_1">
+        <inertial>
+            <origin xyz="-1.6653345369377348e-16 -0.04673529188000056 -2.8160945797495174e-11" rpy="0 0 0"/>
+            <mass value="5.211945183934523"/>
+            <inertia ixx="0.008209" iyy="0.008038" izz="0.004805" ixy="-0.0" iyz="0.0" ixz="-0.0"/>
+        </inertial>
+        <visual>
+            <origin xyz="0.4 0.1925 -0.1625" rpy="0 0 0"/>
+            <geometry>
+                <mesh filename="file://$(find arm_description)/meshes/wrist_1.stl" scale="0.001 0.001 0.001"/>
+            </geometry>
+            <material name="silver"/>
+        </visual>
+        <collision>
+            <origin xyz="0.4 0.1925 -0.1625" rpy="0 0 0"/>
+            <geometry>
+                <mesh filename="file://$(find arm_description)/meshes/wrist_1.stl" scale="0.001 0.001 0.001"/>
+            </geometry>
+        </collision>
+    </link>
+    <joint name="waist_joint" type="revolute">
+        <origin xyz="0.0 0.0 0.115" rpy="0 0 0"/>
         <parent link="base_link"/>
-        <child link="shoulder_mount_1"/>
+        <child link="shoulder_1"/>
         <axis xyz="0.0 0.0 1.0"/>
+        <limit upper="6.265732" lower="0.0" effort="100" velocity="100"/>
     </joint>
     <joint name="shoulder_joint" type="revolute">
-        <origin xyz="-0.0001 0.035 0.0631" rpy="0 0 0"/>
-        <parent link="shoulder_mount_1"/>
-        <child link="shoulder_1"/>
-        <axis xyz="0.0 1.0 0.0"/>
-        <limit upper="3.141593" lower="0.0" effort="100" velocity="100"/>
+        <origin xyz="0.0 -0.0575 0.0475" rpy="0 0 0"/>
+        <parent link="shoulder_1"/>
+        <child link="should_biceptricep_link_1"/>
+        <axis xyz="0.0 -1.0 -0.0"/>
+        <limit upper="6.283185" lower="3.141593" effort="100" velocity="100"/>
+    </joint>
+    <joint name="Rigid 7" type="fixed">
+        <origin xyz="-0.2 -0.02 0.0" rpy="0 0 0"/>
+        <parent link="should_biceptricep_link_1"/>
+        <child link="biceptricep_1"/>
+    </joint>
+    <joint name="biceptricep_joint" type="revolute">
+        <origin xyz="0.0 0.0 0.0" rpy="0 0 0"/>
+        <parent link="biceptricep_1"/>
+        <child link="biceptricep_forearm_link_1"/>
+        <axis xyz="0.0 -1.0 -0.0"/>
+        <limit upper="6.265732" lower="0.0" effort="100" velocity="100"/>
+    </joint>
+    <joint name="Rigid 8" type="fixed">
+        <origin xyz="-0.2 0.0 0.0" rpy="0 0 0"/>
+        <parent link="biceptricep_forearm_link_1"/>
+        <child link="forearm_1"/>
+    </joint>
+    <joint name="forearm_joint" type="continuous">
+        <origin xyz="0.0 -0.115 0.0" rpy="0 0 0"/>
+        <parent link="forearm_1"/>
+        <child link="wrist_1"/>
+        <axis xyz="-0.0 1.0 -0.0"/>
     </joint>
     <link name="world"/>
