Commit message: -6DOF urdf

File: arm_control/urdf/joints.macro.xacro (robot description, xacro)
@@ -2,5 +2,5 @@
 <robot xmlns:xacro="http://www.ros.org/wiki/xacro">
     <xacro:macro name="joints">
-        <joint name="waist_joint">
+        <joint name="joint1">
             <command_interface name="position"/>
             <state_interface name="position">
@@ -8,5 +8,5 @@
             </state_interface>
         </joint>
-        <joint name="shoulder_joint">
+        <joint name="joint2">
             <command_interface name="position"/>
             <state_interface name="position">
@@ -14,5 +14,5 @@
             </state_interface>
         </joint>
-        <joint name="biceptricep_joint">
+        <joint name="joint3">
             <command_interface name="position"/>
             <state_interface name="position">
@@ -20,5 +20,5 @@
             </state_interface>
         </joint>
-        <joint name="forearm_joint">
+        <joint name="joint4">
             <command_interface name="position"/>
             <state_interface name="position">
@@ -26,5 +26,17 @@
             </state_interface>
         </joint>
-        <joint name="wrist_joint">
+        <joint name="joint5">
+            <command_interface name="position"/>
+            <state_interface name="position">
+                <param name="initial_value">0.0</param>
+            </state_interface>
+        </joint>
+        <joint name="joint6">
+            <command_interface name="position"/>
+            <state_interface name="position">
+                <param name="initial_value">0.0</param>
+            </state_interface>
+        </joint>
+        <joint name="joint7">
             <command_interface name="position"/>
             <state_interface name="position">

File: arm_control/urdf/ros2_control.xacro (robot description, xacro)
@@ -2,7 +2,7 @@
 <robot xmlns:xacro="http://www.ros.org/wiki/xacro">
     <xacro:include filename="joints.macro.xacro"/>
-    <ros2_control name="ArmHardware" type="system">
+    <ros2_control name="FakeSystem" type="system">
         <hardware>
-            <plugin>arm_firmware/ArmHardware</plugin>
+            <plugin>mock_components/GenericSystem</plugin>
         </hardware>
         <xacro:joints/>

File: arm_description/urdf/arm_core.xacro (robot description, xacro)
@@ -107,19 +107,59 @@
     <link name="arm_link6_1">
         <inertial>
-            <origin xyz="2.183900666265855e-07 -1.917245794849252e-07 0.005955315753380375" rpy="0 0 0"/>
+            <origin xyz="1.5872838070894908e-05 -0.02828120535039978 0.05185557651993" rpy="0 0 0"/>
+            <mass value="3.055536790464196"/>
+            <inertia ixx="0.003628" iyy="0.003706" izz="0.002737" ixy="0.0" iyz="0.000466" ixz="-0.0"/>
+        </inertial>
+        <visual>
+            <origin xyz="0.000408 -0.000408 -0.526" rpy="0 0 0"/>
+            <geometry>
+                <mesh filename="file://$(find arm_description)/meshes/arm_link6_1.stl" scale="0.001 0.001 0.001"/>
+            </geometry>
+            <material name="silver"/>
+        </visual>
+        <collision>
+            <origin xyz="0.000408 -0.000408 -0.526" rpy="0 0 0"/>
+            <geometry>
+                <mesh filename="file://$(find arm_description)/meshes/arm_link6_1.stl" scale="0.001 0.001 0.001"/>
+            </geometry>
+        </collision>
+    </link>
+    <link name="arm_link7_1">
+        <inertial>
+            <origin xyz="-0.00019611149028537638 0.00634486877981871 0.09901048510996291" rpy="0 0 0"/>
+            <mass value="3.341835621962638"/>
+            <inertia ixx="0.009045" iyy="0.009197" izz="0.002746" ixy="-0.0" iyz="0.000632" ixz="8e-06"/>
+        </inertial>
+        <visual>
+            <origin xyz="0.00039 0.002592 -0.586821" rpy="0 0 0"/>
+            <geometry>
+                <mesh filename="file://$(find arm_description)/meshes/arm_link7_1.stl" scale="0.001 0.001 0.001"/>
+            </geometry>
+            <material name="silver"/>
+        </visual>
+        <collision>
+            <origin xyz="0.00039 0.002592 -0.586821" rpy="0 0 0"/>
+            <geometry>
+                <mesh filename="file://$(find arm_description)/meshes/arm_link7_1.stl" scale="0.001 0.001 0.001"/>
+            </geometry>
+        </collision>
+    </link>
+    <link name="arm_link8_1">
+        <inertial>
+            <origin xyz="3.275850999073793e-07 -2.875868694327899e-07 0.005955315753381596" rpy="0 0 0"/>
             <mass value="0.3239171876105671"/>
-            <inertia ixx="0.000187" iyy="0.000187" izz="0.000369" ixy="0.0" iyz="-0.0" ixz="-0.0"/>
-        </inertial>
-        <visual>
-            <origin xyz="0.000408 -0.000408 -0.526" rpy="0 0 0"/>
-            <geometry>
-                <mesh filename="file://$(find arm_description)/meshes/arm_link6_1.stl" scale="0.001 0.001 0.001"/>
-            </geometry>
-            <material name="silver"/>
-        </visual>
-        <collision>
-            <origin xyz="0.000408 -0.000408 -0.526" rpy="0 0 0"/>
-            <geometry>
-                <mesh filename="file://$(find arm_description)/meshes/arm_link6_1.stl" scale="0.001 0.001 0.001"/>
+            <inertia ixx="0.000187" iyy="0.000187" izz="0.000369" ixy="0.0" iyz="-0.0" ixz="0.0"/>
+        </inertial>
+        <visual>
+            <origin xyz="0.000612 -0.000612 -0.739" rpy="0 0 0"/>
+            <geometry>
+                <mesh filename="file://$(find arm_description)/meshes/arm_link8_1.stl" scale="0.001 0.001 0.001"/>
+            </geometry>
+            <material name="silver"/>
+        </visual>
+        <collision>
+            <origin xyz="0.000612 -0.000612 -0.739" rpy="0 0 0"/>
+            <geometry>
+                <mesh filename="file://$(find arm_description)/meshes/arm_link8_1.stl" scale="0.001 0.001 0.001"/>
             </geometry>
         </collision>
@@ -127,10 +167,10 @@
     <link name="hand_1">
         <inertial>
-            <origin xyz="3.121348217252802e-06 -0.015949144186493007 0.011731923287016999" rpy="0 0 0"/>
-            <mass value="0.11691767429633958"/>
+            <origin xyz="3.2305432505329995e-06 -0.01594924004878426 0.011731923287019663" rpy="0 0 0"/>
+            <mass value="0.11691767429634384"/>
             <inertia ixx="0.000152" iyy="3.2e-05" izz="0.000128" ixy="-0.0" iyz="3.4e-05" ixz="0.0"/>
         </inertial>
         <visual>
-            <origin xyz="0.000408 -0.000408 -0.5365" rpy="0 0 0"/>
+            <origin xyz="0.000612 -0.000612 -0.7495" rpy="0 0 0"/>
             <geometry>
                 <mesh filename="file://$(find arm_description)/meshes/hand_1.stl" scale="0.001 0.001 0.001"/>
@@ -139,5 +179,5 @@
         </visual>
         <collision>
-            <origin xyz="0.000408 -0.000408 -0.5365" rpy="0 0 0"/>
+            <origin xyz="0.000612 -0.000612 -0.7495" rpy="0 0 0"/>
             <geometry>
                 <mesh filename="file://$(find arm_description)/meshes/hand_1.stl" scale="0.001 0.001 0.001"/>
@@ -147,10 +187,10 @@
     <link name="finger_1">
         <inertial>
-            <origin xyz="2.1839006656326808e-07 0.00249980827542038 0.02500000000000191" rpy="0 0 0"/>
-            <mass value="0.03924999999999993"/>
-            <inertia ixx="8e-06" iyy="9e-06" izz="1e-06" ixy="-0.0" iyz="-0.0" ixz="-0.0"/>
-        </inertial>
-        <visual>
-            <origin xyz="0.000408 0.044592 -0.5415" rpy="0 0 0"/>
+            <origin xyz="3.2758509984460397e-07 0.0024997124131302187 0.025000000000003464" rpy="0 0 0"/>
+            <mass value="0.039249999999999986"/>
+            <inertia ixx="8e-06" iyy="9e-06" izz="1e-06" ixy="-0.0" iyz="0.0" ixz="-0.0"/>
+        </inertial>
+        <visual>
+            <origin xyz="0.000612 0.044388 -0.7545" rpy="0 0 0"/>
             <geometry>
                 <mesh filename="file://$(find arm_description)/meshes/finger_1.stl" scale="0.001 0.001 0.001"/>
@@ -159,5 +199,5 @@
         </visual>
         <collision>
-            <origin xyz="0.000408 0.044592 -0.5415" rpy="0 0 0"/>
+            <origin xyz="0.000612 0.044388 -0.7545" rpy="0 0 0"/>
             <geometry>
                 <mesh filename="file://$(find arm_description)/meshes/finger_1.stl" scale="0.001 0.001 0.001"/>
@@ -165,5 +205,5 @@
         </collision>
     </link>
-    <joint name="waist_joint" type="revolute">
+    <joint name="joint1" type="revolute">
         <origin xyz="0.0 0.0 0.1" rpy="0 0 0"/>
         <parent link="base_link"/>
@@ -172,5 +212,5 @@
         <limit lower="-${PI}" upper="${PI}" effort="${effort}" velocity="${velocity}"/>
     </joint>
-    <joint name="shoulder_joint" type="revolute">
+    <joint name="joint2" type="revolute">
         <origin xyz="1.8e-05 -0.003 0.060821" rpy="0 0 0"/>
         <parent link="arm_link2_1"/>
@@ -179,5 +219,5 @@
         <limit lower="-1.833" upper="1.833" effort="${effort}" velocity="${velocity}"/>
     </joint>
-    <joint name="biceptricep_joint" type="revolute">
+    <joint name="joint3" type="revolute">
         <origin xyz="-0.000222 0.003204 0.152179" rpy="0 0 0"/>
         <parent link="arm_link3_1"/>
@@ -186,5 +226,5 @@
         <limit lower="-${PI}" upper="${PI}" effort="${effort}" velocity="${velocity}"/>
     </joint>
-    <joint name="forearm_joint" type="revolute">
+    <joint name="joint4" type="revolute">
         <origin xyz="1.8e-05 -0.003 0.060821" rpy="0 0 0"/>
         <parent link="arm_link4_1"/>
@@ -193,5 +233,5 @@
         <limit lower="-1.833" upper="1.833" effort="${effort}" velocity="${velocity}"/>
     </joint>
-    <joint name="wrist_joint" type="revolute">
+    <joint name="joint5" type="revolute">
         <origin xyz="-0.000222 0.003204 0.152179" rpy="0 0 0"/>
         <parent link="arm_link5_1"/>
@@ -200,14 +240,21 @@
         <limit lower="-${PI}" upper="${PI}" effort="${effort}" velocity="${velocity}"/>
     </joint>
-    <link name="panda_link8" />
-    <joint name="panda_joint8" type="fixed">
-        <origin rpy="0 0 0" xyz="0 0 0.107" />
-        <parent link="arm_link5_1" />
-        <child link="panda_link8" />
-        <axis xyz="0 0 0" />
+    <joint name="joint6" type="revolute">
+        <origin xyz="1.8e-05 -0.003 0.060821" rpy="0 0 0"/>
+        <parent link="arm_link6_1"/>
+        <child link="arm_link7_1"/>
+        <axis xyz="0.0 1.0 0.0"/>
+        <limit lower="-1.833" upper="1.833" effort="${effort}" velocity="${velocity}"/>
+    </joint>
+    <joint name="joint7" type="revolute">
+        <origin xyz="-0.000222 0.003204 0.152179" rpy="0 0 0"/>
+        <parent link="arm_link7_1"/>
+        <child link="arm_link8_1"/>
+        <axis xyz="-0.0 -0.0 1.0"/>
+        <limit lower="-${PI}" upper="${PI}" effort="${effort}" velocity="${velocity}"/>
     </joint>
     <joint name="hand_joint" type="fixed">
         <origin xyz="0.0 0.0 0.0105" rpy="0 0 0"/>
-        <parent link="panda_link8"/>
+        <parent link="arm_link8_1"/>
         <child link="hand_1"/>
     </joint>
