Commit message: joint_1 working on firmware

File: arm_control/urdf/joints.macro.xacro (robot description, xacro)
@@ -2,5 +2,5 @@
 <robot xmlns:xacro="http://www.ros.org/wiki/xacro">
     <xacro:macro name="joints">
-        <joint name="joint1">
+        <joint name="joint_1">
             <command_interface name="position"/>
             <state_interface name="position">
@@ -8,46 +8,10 @@
             </state_interface>
         </joint>
-        <joint name="joint2">
+        <!-- <joint name="finger_joint">
             <command_interface name="position"/>
             <state_interface name="position">
                 <param name="initial_value">0.0</param>
             </state_interface>
-        </joint>
-        <joint name="joint3">
-            <command_interface name="position"/>
-            <state_interface name="position">
-                <param name="initial_value">0.0</param>
-            </state_interface>
-        </joint>
-        <joint name="joint4">
-            <command_interface name="position"/>
-            <state_interface name="position">
-                <param name="initial_value">0.0</param>
-            </state_interface>
-        </joint>
-        <joint name="joint5">
-            <command_interface name="position"/>
-            <state_interface name="position">
-                <param name="initial_value">0.0</param>
-            </state_interface>
-        </joint>
-        <joint name="joint6">
-            <command_interface name="position"/>
-            <state_interface name="position">
-                <param name="initial_value">0.0</param>
-            </state_interface>
-        </joint>
-        <joint name="joint7">
-            <command_interface name="position"/>
-            <state_interface name="position">
-                <param name="initial_value">0.0</param>
-            </state_interface>
-        </joint>
-        <joint name="finger_joint">
-            <command_interface name="position"/>
-            <state_interface name="position">
-                <param name="initial_value">0.0</param>
-            </state_interface>
-        </joint>
+        </joint> -->
     </xacro:macro>
 </robot>

File: arm_description/urdf/arm_core.xacro (robot description, xacro)
@@ -1,268 +1,68 @@
-<?xml version="1.0" ?>
+<?xml version="1.0"?>
 <robot name="arm" xmlns:xacro="http://www.ros.org/wiki/xacro">
-    <xacro:include filename="$(find arm_description)/urdf/materials.xacro"/>
-    <xacro:property name="PI" value="3.14159265359"/>
-    <xacro:property name="effort" value="30"/>
-    <xacro:property name="velocity" value="10"/>
+    <xacro:include filename="$(find arm_description)/urdf/materials.xacro" />
+    <xacro:include filename="$(find arm_description)/urdf/arm.trans" />
+    <xacro:property name="PI" value="3.14159265359" />
+    <xacro:property name="effort" value="30" />
+    <xacro:property name="velocity" value="10" />
+    <link name="world" />
     <link name="base_link">
         <inertial>
-            <origin xyz="0.0 0.0 0.04999999999999999" rpy="0 0 0"/>
-            <mass value="4.454483858479053"/>
-            <inertia ixx="0.005724" iyy="0.005724" izz="0.004023" ixy="-0.0" iyz="0.0" ixz="0.0"/>
+            <origin xyz="-7.122570585896167e-18 -7.122570585896167e-18 0.0115" rpy="0 0 0" />
+            <mass value="1.2529769489148532" />
+            <inertia ixx="0.000747" iyy="0.000747" izz="0.001384" ixy="-0.0" iyz="-0.0" ixz="-0.0" />
         </inertial>
         <visual>
-            <origin xyz="0 0 0" rpy="0 0 0"/>
+            <origin xyz="0 0 0" rpy="0 0 0" />
             <geometry>
-                <mesh filename="file://$(find arm_description)/meshes/base_link.stl" scale="0.001 0.001 0.001"/>
+                <mesh filename="file://$(find arm_description)/meshes/base_link.stl"
+                    scale="0.001 0.001 0.001" />
             </geometry>
-            <material name="silver"/>
+            <material name="silver" />
         </visual>
         <collision>
-            <origin xyz="0 0 0" rpy="0 0 0"/>
+            <origin xyz="0 0 0" rpy="0 0 0" />
             <geometry>
-                <mesh filename="file://$(find arm_description)/meshes/base_link.stl" scale="0.001 0.001 0.001"/>
+                <mesh filename="file://$(find arm_description)/meshes/base_link.stl"
+                    scale="0.001 0.001 0.001" />
             </geometry>
         </collision>
     </link>
-    <link name="arm_link2_1">
+    <!-- base_joint fixes base_link to the environment -->
+    <joint name="base_joint" type="fixed">
+        <parent link="world" />
+        <child link="base_link" />
+        <origin xyz="0 0 0" rpy="0 0 0" />
+        <axis xyz="0 0 1" />
+    </joint>
+    <link name="link_1_1">
         <inertial>
-            <origin xyz="1.5654448004331833e-05 -0.02828101362582021 0.05185557651992784" rpy="0 0 0"/>
-            <mass value="3.055536790464196"/>
-            <inertia ixx="0.003628" iyy="0.003706" izz="0.002737" ixy="0.0" iyz="0.000466" ixz="-0.0"/>
+            <origin xyz="1.0865459766237383e-16 1.9984014443252817e-17 0.042728114320090264"
+                rpy="0 0 0" />
+            <mass value="1.4164963986999342" />
+            <inertia ixx="0.000964" iyy="0.001818" izz="0.000979" ixy="-0.0" iyz="-0.0" ixz="-0.0" />
         </inertial>
         <visual>
-            <origin xyz="-0.0 -0.0 -0.1" rpy="0 0 0"/>
+            <origin xyz="-0.0 -0.0 -0.023" rpy="0 0 0" />
             <geometry>
-                <mesh filename="file://$(find arm_description)/meshes/arm_link2_1.stl" scale="0.001 0.001 0.001"/>
+                <mesh filename="file://$(find arm_description)/meshes/link_1_1.stl"
+                    scale="0.001 0.001 0.001" />
             </geometry>
-            <material name="silver"/>
+            <material name="silver" />
         </visual>
         <collision>
-            <origin xyz="-0.0 -0.0 -0.1" rpy="0 0 0"/>
+            <origin xyz="-0.0 -0.0 -0.023" rpy="0 0 0" />
             <geometry>
-                <mesh filename="file://$(find arm_description)/meshes/arm_link2_1.stl" scale="0.001 0.001 0.001"/>
+                <mesh filename="file://$(find arm_description)/meshes/link_1_1.stl"
+                    scale="0.001 0.001 0.001" />
             </geometry>
         </collision>
     </link>
-    <link name="arm_link3_1">
-        <inertial>
-            <origin xyz="-0.00019632988035193946 0.006345060504398406 0.09901048510996069" rpy="0 0 0"/>
-            <mass value="3.341835621962638"/>
-            <inertia ixx="0.009045" iyy="0.009197" izz="0.002746" ixy="-0.0" iyz="0.000632" ixz="8e-06"/>
-        </inertial>
-        <visual>
-            <origin xyz="-1.8e-05 0.003 -0.160821" rpy="0 0 0"/>
-            <geometry>
-                <mesh filename="file://$(find arm_description)/meshes/arm_link3_1.stl" scale="0.001 0.001 0.001"/>
-            </geometry>
-            <material name="silver"/>
-        </visual>
-        <collision>
-            <origin xyz="-1.8e-05 0.003 -0.160821" rpy="0 0 0"/>
-            <geometry>
-                <mesh filename="file://$(find arm_description)/meshes/arm_link3_1.stl" scale="0.001 0.001 0.001"/>
-            </geometry>
-        </collision>
-    </link>
-    <link name="arm_link4_1">
-        <inertial>
-            <origin xyz="1.576364303761414e-05 -0.028281109488109926 0.05185557651992889" rpy="0 0 0"/>
-            <mass value="3.055536790464196"/>
-            <inertia ixx="0.003628" iyy="0.003706" izz="0.002737" ixy="0.0" iyz="0.000466" ixz="-0.0"/>
-        </inertial>
-        <visual>
-            <origin xyz="0.000204 -0.000204 -0.313" rpy="0 0 0"/>
-            <geometry>
-                <mesh filename="file://$(find arm_description)/meshes/arm_link4_1.stl" scale="0.001 0.001 0.001"/>
-            </geometry>
-            <material name="silver"/>
-        </visual>
-        <collision>
-            <origin xyz="0.000204 -0.000204 -0.313" rpy="0 0 0"/>
-            <geometry>
-                <mesh filename="file://$(find arm_description)/meshes/arm_link4_1.stl" scale="0.001 0.001 0.001"/>
-            </geometry>
-        </collision>
-    </link>
-    <link name="arm_link5_1">
-        <inertial>
-            <origin xyz="-0.00019622068531865714 0.006344964642108612 0.09901048510996169" rpy="0 0 0"/>
-            <mass value="3.341835621962638"/>
-            <inertia ixx="0.009045" iyy="0.009197" izz="0.002746" ixy="-0.0" iyz="0.000632" ixz="8e-06"/>
-        </inertial>
-        <visual>
-            <origin xyz="0.000186 0.002796 -0.373821" rpy="0 0 0"/>
-            <geometry>
-                <mesh filename="file://$(find arm_description)/meshes/arm_link5_1.stl" scale="0.001 0.001 0.001"/>
-            </geometry>
-            <material name="silver"/>
-        </visual>
-        <collision>
-            <origin xyz="0.000186 0.002796 -0.373821" rpy="0 0 0"/>
-            <geometry>
-                <mesh filename="file://$(find arm_description)/meshes/arm_link5_1.stl" scale="0.001 0.001 0.001"/>
-            </geometry>
-        </collision>
-    </link>
-    <link name="arm_link6_1">
-        <inertial>
-            <origin xyz="1.5872838070894908e-05 -0.02828120535039978 0.05185557651993" rpy="0 0 0"/>
-            <mass value="3.055536790464196"/>
-            <inertia ixx="0.003628" iyy="0.003706" izz="0.002737" ixy="0.0" iyz="0.000466" ixz="-0.0"/>
-        </inertial>
-        <visual>
-            <origin xyz="0.000408 -0.000408 -0.526" rpy="0 0 0"/>
-            <geometry>
-                <mesh filename="file://$(find arm_description)/meshes/arm_link6_1.stl" scale="0.001 0.001 0.001"/>
-            </geometry>
-            <material name="silver"/>
-        </visual>
-        <collision>
-            <origin xyz="0.000408 -0.000408 -0.526" rpy="0 0 0"/>
-            <geometry>
-                <mesh filename="file://$(find arm_description)/meshes/arm_link6_1.stl" scale="0.001 0.001 0.001"/>
-            </geometry>
-        </collision>
-    </link>
-    <link name="arm_link7_1">
-        <inertial>
-            <origin xyz="-0.00019611149028537638 0.00634486877981871 0.09901048510996291" rpy="0 0 0"/>
-            <mass value="3.341835621962638"/>
-            <inertia ixx="0.009045" iyy="0.009197" izz="0.002746" ixy="-0.0" iyz="0.000632" ixz="8e-06"/>
-        </inertial>
-        <visual>
-            <origin xyz="0.00039 0.002592 -0.586821" rpy="0 0 0"/>
-            <geometry>
-                <mesh filename="file://$(find arm_description)/meshes/arm_link7_1.stl" scale="0.001 0.001 0.001"/>
-            </geometry>
-            <material name="silver"/>
-        </visual>
-        <collision>
-            <origin xyz="0.00039 0.002592 -0.586821" rpy="0 0 0"/>
-            <geometry>
-                <mesh filename="file://$(find arm_description)/meshes/arm_link7_1.stl" scale="0.001 0.001 0.001"/>
-            </geometry>
-        </collision>
-    </link>
-    <link name="arm_link8_1">
-        <inertial>
-            <origin xyz="3.275850999073793e-07 -2.875868694327899e-07 0.005955315753381596" rpy="0 0 0"/>
-            <mass value="0.3239171876105671"/>
-            <inertia ixx="0.000187" iyy="0.000187" izz="0.000369" ixy="0.0" iyz="-0.0" ixz="0.0"/>
-        </inertial>
-        <visual>
-            <origin xyz="0.000612 -0.000612 -0.739" rpy="0 0 0"/>
-            <geometry>
-                <mesh filename="file://$(find arm_description)/meshes/arm_link8_1.stl" scale="0.001 0.001 0.001"/>
-            </geometry>
-            <material name="silver"/>
-        </visual>
-        <collision>
-            <origin xyz="0.000612 -0.000612 -0.739" rpy="0 0 0"/>
-            <geometry>
-                <mesh filename="file://$(find arm_description)/meshes/arm_link8_1.stl" scale="0.001 0.001 0.001"/>
-            </geometry>
-        </collision>
-    </link>
-    <link name="hand_1">
-        <inertial>
-            <origin xyz="3.2305432505329995e-06 -0.01594924004878426 0.011731923287019663" rpy="0 0 0"/>
-            <mass value="0.11691767429634384"/>
-            <inertia ixx="0.000152" iyy="3.2e-05" izz="0.000128" ixy="-0.0" iyz="3.4e-05" ixz="0.0"/>
-        </inertial>
-        <visual>
-            <origin xyz="0.000612 -0.000612 -0.7495" rpy="0 0 0"/>
-            <geometry>
-                <mesh filename="file://$(find arm_description)/meshes/hand_1.stl" scale="0.001 0.001 0.001"/>
-            </geometry>
-            <material name="silver"/>
-        </visual>
-        <collision>
-            <origin xyz="0.000612 -0.000612 -0.7495" rpy="0 0 0"/>
-            <geometry>
-                <mesh filename="file://$(find arm_description)/meshes/hand_1.stl" scale="0.001 0.001 0.001"/>
-            </geometry>
-        </collision>
-    </link>
-    <link name="finger_1">
-        <inertial>
-            <origin xyz="3.2758509984460397e-07 0.0024997124131302187 0.025000000000003464" rpy="0 0 0"/>
-            <mass value="0.039249999999999986"/>
-            <inertia ixx="8e-06" iyy="9e-06" izz="1e-06" ixy="-0.0" iyz="0.0" ixz="-0.0"/>
-        </inertial>
-        <visual>
-            <origin xyz="0.000612 0.044388 -0.7545" rpy="0 0 0"/>
-            <geometry>
-                <mesh filename="file://$(find arm_description)/meshes/finger_1.stl" scale="0.001 0.001 0.001"/>
-            </geometry>
-            <material name="silver"/>
-        </visual>
-        <collision>
-            <origin xyz="0.000612 0.044388 -0.7545" rpy="0 0 0"/>
-            <geometry>
-                <mesh filename="file://$(find arm_description)/meshes/finger_1.stl" scale="0.001 0.001 0.001"/>
-            </geometry>
-        </collision>
-    </link>
-    <joint name="joint1" type="revolute">
-        <origin xyz="0.0 0.0 0.1" rpy="0 0 0"/>
-        <parent link="base_link"/>
-        <child link="arm_link2_1"/>
-        <axis xyz="0.0 0.0 1.0"/>
-        <limit lower="-${PI}" upper="${PI}" effort="${effort}" velocity="${velocity}"/>
-    </joint>
-    <joint name="joint2" type="revolute">
-        <origin xyz="1.8e-05 -0.003 0.060821" rpy="0 0 0"/>
-        <parent link="arm_link2_1"/>
-        <child link="arm_link3_1"/>
-        <axis xyz="0.0 1.0 0.0"/>
-        <limit lower="-1.833" upper="1.833" effort="${effort}" velocity="${velocity}"/>
-    </joint>
-    <joint name="joint3" type="revolute">
-        <origin xyz="-0.000222 0.003204 0.152179" rpy="0 0 0"/>
-        <parent link="arm_link3_1"/>
-        <child link="arm_link4_1"/>
-        <axis xyz="0.0 -0.0 1.0"/>
-        <limit lower="-${PI}" upper="${PI}" effort="${effort}" velocity="${velocity}"/>
-    </joint>
-    <joint name="joint4" type="revolute">
-        <origin xyz="1.8e-05 -0.003 0.060821" rpy="0 0 0"/>
-        <parent link="arm_link4_1"/>
-        <child link="arm_link5_1"/>
-        <axis xyz="0.0 1.0 0.0"/>
-        <limit lower="-1.833" upper="1.833" effort="${effort}" velocity="${velocity}"/>
-    </joint>
-    <joint name="joint5" type="revolute">
-        <origin xyz="-0.000222 0.003204 0.152179" rpy="0 0 0"/>
-        <parent link="arm_link5_1"/>
-        <child link="arm_link6_1"/>
-        <axis xyz="0.0 -0.0 1.0"/>
-        <limit lower="-${PI}" upper="${PI}" effort="${effort}" velocity="${velocity}"/>
-    </joint>
-    <joint name="joint6" type="revolute">
-        <origin xyz="1.8e-05 -0.003 0.060821" rpy="0 0 0"/>
-        <parent link="arm_link6_1"/>
-        <child link="arm_link7_1"/>
-        <axis xyz="0.0 1.0 0.0"/>
-        <limit lower="-1.833" upper="1.833" effort="${effort}" velocity="${velocity}"/>
-    </joint>
-    <joint name="joint7" type="revolute">
-        <origin xyz="-0.000222 0.003204 0.152179" rpy="0 0 0"/>
-        <parent link="arm_link7_1"/>
-        <child link="arm_link8_1"/>
-        <axis xyz="-0.0 -0.0 1.0"/>
-        <limit lower="-${PI}" upper="${PI}" effort="${effort}" velocity="${velocity}"/>
-    </joint>
-    <joint name="hand_joint" type="fixed">
-        <origin xyz="0.0 0.0 0.0105" rpy="0 0 0"/>
-        <parent link="arm_link8_1"/>
-        <child link="hand_1"/>
-    </joint>
-    <joint name="finger_joint" type="prismatic">
-        <origin xyz="0.0 -0.045 0.005" rpy="0 0 0"/>
-        <parent link="hand_1"/>
-        <child link="finger_1"/>
-        <axis xyz="0.0 -1.0 -0.0"/>
-        <limit upper="0.0" lower="-0.09" effort="100" velocity="100"/>
+    <joint name="joint_1" type="revolute">
+        <origin xyz="0.0 0.0 0.023" rpy="0 0 0" />
+        <parent link="base_link" />
+        <child link="link_1_1" />
+        <axis xyz="0.0 0.0 1.0" />
+        <limit lower="-${PI}" upper="${PI}" effort="${effort}" velocity="${velocity}" />
     </joint>
 </robot>
